File: electronics/autopilot/autopilot.kicad_pcb (KiCad board)
At the start: 2 copper layers, 100.1 x 84.6 mm, 25 parts, among them J1 Conn_01x03_Male, J10 Conn_01x03_Female, J11 Debug, J2 Conn_01x03_Male, J3 Conn_01x03_Male, J4 Conn_01x03_Male, J5 Conn_01x02_Female, J6 GSM_MODULE, J7 IBUS, J8 Screw_Terminal_01x02, J9 Conn_01x08_Female, U1 Pico, U2 SIM28ML, U3 NRF24L01_Breakout, U4 74HC244

Commit message: autopilot board  finished
Parts:
- added L1: 27n, Inductor_SMD:L_1210_3225Metric_Pad1.42x2.65mm_HandSolder, F.Cu at (23.1, 65.5)
- added R6: 10, Resistor_SMD:R_1206_3216Metric_Pad1.30x1.75mm_HandSolder, F.Cu at (23.1, 68.8)
- J1, J2, J3, J4: value Conn_01x03_Male -> SERVO
- J5: value Conn_01x02_Female -> ESC
- J8: value Screw_Terminal_01x02 -> 5V IN
- J9: value Conn_01x08_Female -> IMU
- moved J4 100.8 mm to (77.7, 129.8), turned to -90 degrees
- moved J3 90.0 mm to (77.7, 126.0), turned to -90 degrees
- moved J2 78.8 mm to (77.7, 122.2), turned to -90 degrees
- moved J1 69.6 mm to (77.7, 118.4), turned to -90 degrees
- moved J5 52.5 mm to (52.8, 122.7)
- moved J7 22.9 mm to (49.0, 117.3), turned to -90 degrees
- moved J9 22.1 mm to (42.9, 93.5)
- moved C1 13.5 mm to (42.9, 67.3), turned to -90 degrees
- moved AE1 12.2 mm to (23.1, 72.1)
- moved R2 11.5 mm to (49.5, 111.8), turned to 90 degrees
- moved D1 11.4 mm to (79.5, 95.5)
- moved J8 10.2 mm to (79.8, 67.6), turned to -90 degrees
- moved R1 9.81 mm to (45.2, 113.3)
- moved C2 9.77 mm to (40.1, 67.3), turned to -90 degrees
- moved J6 6.66 mm to (40.4, 106.9), turned to 0 degrees
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Connections:
- U2 pad 14: unconnected-(U2-Pad14) -> Net-(U2-Pad14)
Routing:
- net GND: track 0.00 -> 271.1 mm
- net +3.3V: track 0.00 -> 199.9 mm, vias 0 -> 8
- net +5V: track 0.00 -> 118.6 mm
- net /GPS_RST: track 0.00 -> 65.6 mm, vias 0 -> 2
- net /GSM_RX: track 0.00 -> 40.2 mm
- net /GSM_TX: track 0.00 -> 34.7 mm
- net /PWM_ESC: track 0.00 -> 29.0 mm, vias 0 -> 2
- net /PWM_SERVO2: track 0.00 -> 27.3 mm
- net /PWM_SERVO1: track 0.00 -> 27.1 mm
- net /PWM_SERVO3: track 0.00 -> 25.3 mm
- net /CSN: track 0.00 -> 23.9 mm, vias 0 -> 1
- net /PWM_SERVO4: track 0.00 -> 23.9 mm
- net /MOSI: track 0.00 -> 23.6 mm, vias 0 -> 1
- net /IMU_I2C_SCL: track 0.00 -> 15.3 mm
- net /IMU_I2C_SDA: track 0.00 -> 14.5 mm
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Other:
- board size 100.1 x 84.6 mm -> 70.4 x 68.8 mm

Commit message: minor fixes
Parts:
- moved J5 76.4 mm to (128.3, 134.5)
- moved U3 76.4 mm to (159.3, 117.5)
- moved AE1 76.4 mm to (98.6, 83.9)
- moved C1 76.4 mm to (118.4, 79.1)
- moved D1 76.4 mm to (154.9, 107.3)
- moved J1 76.4 mm to (153.2, 130.2)
- moved J9 76.4 mm to (118.4, 105.3)
- moved L1 76.4 mm to (98.6, 77.3)
- moved R1 76.4 mm to (120.7, 125.1)
- moved R2 76.4 mm to (125.0, 123.6)
- moved R5 76.4 mm to (154.9, 109.9)
- moved R6 76.4 mm to (98.6, 80.6)
- moved U1 76.4 mm to (139.4, 101.0)
- moved C2 76.4 mm to (115.6, 79.1)
- moved C3 76.4 mm to (160.5, 113.9)
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
Commit message: autopilot finished secend version
Parts:
- J10: value Conn_01x03_Female -> MPPT_I2C
Routing:
- net GND: track 271.1 -> 91.0 mm, vias 0 -> 10
- net +5V: track 118.6 -> 146.6 mm
- net /MPPT_I2C_SDA: track 0.00 -> 6.71 mm
- net /MPPT_I2C_SCL: track 0.00 -> 6.71 mm
- net +3.3V: track 199.9 -> 199.7 mm, vias 8 -> 6
- added copper zone on B.Cu, net GND

Commit message: power board schematic almost finished
Parts:
- added J12: 5V IN, moje:ARK, F.Cu at (155.2, 89.0)
Connections:
- U1 pad 36: +3.3V -> unconnected-(U1-Pad36)
Routing:
- net +3.3V: track 199.7 -> 190.9 mm
Changed lines of the file:
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@@
   (net 65 "/LED")
   (net 66 "Net-(L1-Pad1)")
+  (net 67 "unconnected-(U1-Pad36)")
   (footprint "Connector_PinHeader_2.54mm:PinHeader_1x02_P2.54mm_Vertical" (layer "F.Cu")
     (at 128.27 134.488)
@@
       (rotate (xyz 0 0 0))
     )
+  )
+  (footprint "moje:ARK" (layer "F.Cu")
+    (at 155.194 89.027 90)
+    (property "Sheetfile" "autopilot.kicad_sch")
+    (property "Sheetname" "")
+    (attr through_hole)
+    (fp_text reference "J12" (at 0 -0.5 90 unlocked) (layer "F.SilkS")
+      (effects (font (size 1 1) (thickness 0.15)))
+    )
+    (fp_text value "5V IN" (at 0 1 90 unlocked) (layer "F.Fab")
+      (effects (font (size 1 1) (thickness 0.15)))
+    )
+    (fp_text user "${REFERENCE}" (at 0 2.5 90 unlocked) (layer "F.Fab")
+      (effects (font (size 1 1) (thickness 0.15)))
+    )
+    (pad "1" thru_hole oval (at -2.54 0 90) (size 1.5 3) (drill 0.762) (layers *.Cu *.Mask)
+      (net 2 "+3.3V") (pinfunction "Pin_1") (pintype "passive"))
+    (pad "2" thru_hole oval (at 2.54 0 90) (size 1.5 3) (drill 0.762) (layers *.Cu *.Mask)
+      (net 3 "GND") (pinfunction "Pin_2") (pintype "passive"))
   )
   (footprint "Capacitor_SMD:C_1206_3216Metric_Pad1.33x1.80mm_HandSolder" (layer "F.Cu")
@@
       (net 43 "unconnected-(U1-Pad35)") (pinfunction "ADC_VREF") (pintype "power_in"))
     (pad "36" smd rect (at 8.89 -13.97) (size 3.5 1.7) (drill (offset 0.9 0)) (layers "F.Cu" "F.Mask")
-      (net 2 "+3.3V") (pinfunction "3V3") (pintype "power_in"))
+      (net 67 "unconnected-(U1-Pad36)") (pinfunction "3V3") (pintype "power_in"))
     (pad "36" thru_hole oval (at 8.89 -13.97) (size 1.7 1.7) (drill 1.02) (layers *.Cu *.Mask)
-      (net 2 "+3.3V") (pinfunction "3V3") (pintype "power_in"))
+      (net 67 "unconnected-(U1-Pad36)") (pinfunction "3V3") (pintype "power_in"))
     (pad "37" thru_hole oval (at 8.89 -16.51) (size 1.7 1.7) (drill 1.02) (layers *.Cu *.Mask)
       (net 44 "unconnected-(U1-Pad37)") (pinfunction "3V3_EN") (pintype "input"))
@@
   (segment (start 165.1255 116.954) (end 165.1255 131.6735) (width 0.35) (layer "F.Cu") (net 2))
   (segment (start 165.1255 131.6735) (end 164.338 132.461) (width 0.35) (layer "F.Cu") (net 2))
-  (segment (start 155.956 86.995) (end 148.336 86.995) (width 0.35) (layer "F.Cu") (net 2))
   (segment (start 118.364 77.5585) (end 118.364 76.073) (width 0.35) (layer "F.Cu") (net 2))
+  (segment (start 155.194 91.567) (end 160.528 91.567) (width 0.5) (layer "F.Cu") (net 2))
   (segment (start 115.3565 77.345) (end 115.57 77.5585) (width 0.35) (layer "F.Cu") (net 2))
   (segment (start 117.094 92.583) (end 118.364 92.583) (width 0.35) (layer "F.Cu") (net 2))
@@
   (segment (start 162.0905 113.919) (end 162.0905 93.1295) (width 0.35) (layer "F.Cu") (net 2))
   (segment (start 118.364 76.073) (end 119.126 75.311) (width 0.35) (layer "F.Cu") (net 2))
-  (segment (start 162.0905 93.1295) (end 155.956 86.995) (width 0.35) (layer "F.Cu") (net 2))
   (segment (start 118.364 102.743) (end 116.586 102.743) (width 0.35) (layer "F.Cu") (net 2))
   (segment (start 141.478 142.875) (end 123.19 142.875) (width 0.35) (layer "F.Cu") (net 2))
@@
   (segment (start 161.798 117.475) (end 161.798 114.2115) (width 0.35) (layer "F.Cu") (net 2))
   (segment (start 116.078 102.235) (end 116.078 93.599) (width 0.35) (layer "F.Cu") (net 2))
+  (segment (start 160.528 91.567) (end 162.0905 93.1295) (width 0.5) (layer "F.Cu") (net 2))
   (via (at 118.14 137.825) (size 0.8) (drill 0.4) (layers "F.Cu" "B.Cu") (net 2))
   (via (at 118.237 123.444) (size 0.8) (drill 0.4) (layers "F.Cu" "B.Cu") (net 2))

Commit message: autopilot board minor fixes
Parts:
- added J13: Vbatt, Connector_PinHeader_2.54mm:PinHeader_1x02_P2.54mm_Vertical, F.Cu at (158.2, 92.1)
- moved J12 16.0 mm to (162.1, 103.5)
Connections:
- U1 pad 34: unconnected-(U1-Pad34) -> Net-(U1-Pad34)
Routing:
- net +3.3V: track 190.9 -> 170.8 mm
- net Net-(U1-Pad34): track 0.00 -> 9.91 mm
- net GND: track 91.0 -> 100.2 mm
Changed lines of the file:
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@@
   (net 40 "unconnected-(U1-Pad31)")
   (net 41 "unconnected-(U1-Pad32)")
-  (net 42 "unconnected-(U1-Pad34)")
+  (net 42 "Net-(U1-Pad34)")
   (net 43 "unconnected-(U1-Pad35)")
   (net 44 "unconnected-(U1-Pad37)")
@@
       (net 22 "/IBUS") (pintype "passive"))
     (model "${KICAD6_3DMODEL_DIR}/Resistor_SMD.3dshapes/R_1206_3216Metric.wrl"
+      (offset (xyz 0 0 0))
+      (scale (xyz 1 1 1))
+      (rotate (xyz 0 0 0))
+    )
+  )
+  (footprint "Connector_PinHeader_2.54mm:PinHeader_1x02_P2.54mm_Vertical" (layer "F.Cu")
+    (at 158.242 92.07)
+    (descr "Through hole straight pin header, 1x02, 2.54mm pitch, single row")
+    (tags "Through hole pin header THT 1x02 2.54mm single row")
+    (property "Sheetfile" "autopilot.kicad_sch")
+    (property "Sheetname" "")
+    (attr through_hole)
+    (fp_text reference "J13" (at 0 -2.33) (layer "F.SilkS")
+      (effects (font (size 1 1) (thickness 0.15)))
+    )
+    (fp_text value "Vbatt" (at 0 4.87) (layer "F.Fab")
+      (effects (font (size 1 1) (thickness 0.15)))
+    )
+    (fp_text user "${REFERENCE}" (at 0 1.27 90) (layer "F.Fab")
+      (effects (font (size 1 1) (thickness 0.15)))
+    )
+    (fp_line (start -1.33 -1.33) (end 0 -1.33) (layer "F.SilkS") (width 0.12))
+    (fp_line (start -1.33 1.27) (end 1.33 1.27) (layer "F.SilkS") (width 0.12))
+    (fp_line (start 1.33 1.27) (end 1.33 3.87) (layer "F.SilkS") (width 0.12))
+    (fp_line (start -1.33 0) (end -1.33 -1.33) (layer "F.SilkS") (width 0.12))
+    (fp_line (start -1.33 3.87) (end 1.33 3.87) (layer "F.SilkS") (width 0.12))
+    (fp_line (start -1.33 1.27) (end -1.33 3.87) (layer "F.SilkS") (width 0.12))
+    (fp_line (start -1.8 -1.8) (end -1.8 4.35) (layer "F.CrtYd") (width 0.05))
+    (fp_line (start 1.8 4.35) (end 1.8 -1.8) (layer "F.CrtYd") (width 0.05))
+    (fp_line (start -1.8 4.35) (end 1.8 4.35) (layer "F.CrtYd") (width 0.05))
+    (fp_line (start 1.8 -1.8) (end -1.8 -1.8) (layer "F.CrtYd") (width 0.05))
+    (fp_line (start -1.27 -0.635) (end -0.635 -1.27) (layer "F.Fab") (width 0.1))
+    (fp_line (start 1.27 3.81) (end -1.27 3.81) (layer "F.Fab") (width 0.1))
+    (fp_line (start -0.635 -1.27) (end 1.27 -1.27) (layer "F.Fab") (width 0.1))
+    (fp_line (start -1.27 3.81) (end -1.27 -0.635) (layer "F.Fab") (width 0.1))
+    (fp_line (start 1.27 -1.27) (end 1.27 3.81) (layer "F.Fab") (width 0.1))
+    (pad "1" thru_hole rect (at 0 0) (size 1.7 1.7) (drill 1) (layers *.Cu *.Mask)
+      (net 42 "Net-(U1-Pad34)") (pinfunction "Pin_1") (pintype "passive"))
+    (pad "2" thru_hole oval (at 0 2.54) (size 1.7 1.7) (drill 1) (layers *.Cu *.Mask)
+      (net 3 "GND") (pinfunction "Pin_2") (pintype "passive"))
+    (model "${KICAD6_3DMODEL_DIR}/Connector_PinHeader_2.54mm.3dshapes/PinHeader_1x02_P2.54mm_Vertical.wrl"
       (offset (xyz 0 0 0))
       (scale (xyz 1 1 1))
@@
   )
   (footprint "moje:ARK" (layer "F.Cu")
-    (at 155.194 89.027 90)
+    (at 162.052 103.505 90)
     (property "Sheetfile" "autopilot.kicad_sch")
     (property "Sheetname" "")
@@
       (net 3 "GND") (pinfunction "AGND") (pintype "power_in"))
     (pad "34" thru_hole oval (at 8.89 -8.89) (size 1.7 1.7) (drill 1.02) (layers *.Cu *.Mask)
-      (net 42 "unconnected-(U1-Pad34)") (pinfunction "GPIO28_ADC2") (pintype "bidirectional"))
+      (net 42 "Net-(U1-Pad34)") (pinfunction "GPIO28_ADC2") (pintype "bidirectional"))
     (pad "34" smd rect (at 8.89 -8.89) (size 3.5 1.7) (drill (offset 0.9 0)) (layers "F.Cu" "F.Mask")
-      (net 42 "unconnected-(U1-Pad34)") (pinfunction "GPIO28_ADC2") (pintype "bidirectional"))
+      (net 42 "Net-(U1-Pad34)") (pinfunction "GPIO28_ADC2") (pintype "bidirectional"))
     (pad "35" thru_hole oval (at 8.89 -11.43) (size 1.7 1.7) (drill 1.02) (layers *.Cu *.Mask)
       (net 43 "unconnected-(U1-Pad35)") (pinfunction "ADC_VREF") (pintype "power_in"))
@@
   (segment (start 116.586 102.743) (end 116.078 102.235) (width 0.35) (layer "F.Cu") (net 2))
   (segment (start 162.0905 113.919) (end 165.1255 116.954) (width 0.35) (layer "F.Cu") (net 2))
+  (segment (start 162.052 108.204) (end 162.56 108.712) (width 0.5) (layer "F.Cu") (net 2))
+  (segment (start 162.052 106.045) (end 162.052 108.204) (width 0.5) (layer "F.Cu") (net 2))
+  (segment (start 162.56 113.4495) (end 162.0905 113.919) (width 0.5) (layer "F.Cu") (net 2))
   (segment (start 118.364 77.5585) (end 115.57 77.5585) (width 0.35) (layer "F.Cu") (net 2))
   (segment (start 162.0905 113.157) (end 161.752 113.4955) (width 0.35) (layer "F.Cu") (net 2))
@@
   (segment (start 123.19 142.875) (end 118.14 137.825) (width 0.35) (layer "F.Cu") (net 2))
   (segment (start 118.237 123.444) (end 116.2 123.444) (width 0.35) (layer "F.Cu") (net 2))
+  (segment (start 162.56 108.712) (end 162.56 113.4495) (width 0.5) (layer "F.Cu") (net 2))
   (segment (start 116.078 93.599) (end 117.094 92.583) (width 0.35) (layer "F.Cu") (net 2))
   (segment (start 164.338 135.763) (end 157.226 142.875) (width 0.35) (layer "F.Cu") (net 2))
@@
   (segment (start 165.1255 131.6735) (end 164.338 132.461) (width 0.35) (layer "F.Cu") (net 2))
   (segment (start 118.364 77.5585) (end 118.364 76.073) (width 0.35) (layer "F.Cu") (net 2))
-  (segment (start 155.194 91.567) (end 160.528 91.567) (width 0.5) (layer "F.Cu") (net 2))
   (segment (start 115.3565 77.345) (end 115.57 77.5585) (width 0.35) (layer "F.Cu") (net 2))
   (segment (start 117.094 92.583) (end 118.364 92.583) (width 0.35) (layer "F.Cu") (net 2))
   (segment (start 116.2 123.444) (end 115.824 123.82) (width 0.35) (layer "F.Cu") (net 2))
-  (segment (start 162.0905 113.919) (end 162.0905 93.1295) (width 0.35) (layer "F.Cu") (net 2))
   (segment (start 118.364 76.073) (end 119.126 75.311) (width 0.35) (layer "F.Cu") (net 2))
   (segment (start 118.364 102.743) (end 116.586 102.743) (width 0.35) (layer "F.Cu") (net 2))
@@
   (segment (start 161.798 117.475) (end 161.798 114.2115) (width 0.35) (layer "F.Cu") (net 2))
   (segment (start 116.078 102.235) (end 116.078 93.599) (width 0.35) (layer "F.Cu") (net 2))
-  (segment (start 160.528 91.567) (end 162.0905 93.1295) (width 0.5) (layer "F.Cu") (net 2))
   (via (at 118.14 137.825) (size 0.8) (drill 0.4) (layers "F.Cu" "B.Cu") (net 2))
   (via (at 118.237 123.444) (size 0.8) (drill 0.4) (layers "F.Cu" "B.Cu") (net 2))
@@
   (segment (start 135.89 138.617) (end 132.775 138.617) (width 0.5) (layer "F.Cu") (net 3))
   (segment (start 126.974 120.015) (end 124.968 122.021) (width 0.5) (layer "F.Cu") (net 3))
+  (segment (start 162.052 100.965) (end 159.893 100.965) (width 0.5) (layer "F.Cu") (net 3))
   (segment (start 132.775 138.617) (end 131.826 137.668) (width 0.5) (layer "F.Cu") (net 3))
   (segment (start 137.354 138.617) (end 135.89 138.617) (width 0.35) (layer "F.Cu") (net 3))
@@
   (segment (start 131.826 137.668) (end 131.186 137.028) (width 0.5) (layer "F.Cu") (net 3))
   (segment (start 135.89 132.767) (end 135.942 132.715) (width 0.35) (layer "F.Cu") (net 3))
+  (segment (start 158.242 94.61) (end 158.242 99.314) (width 0.5) (layer "F.Cu") (net 3))
   (segment (start 159.258 114.2115) (end 158.9655 113.919) (width 0.5) (layer "F.Cu") (net 3))
   (segment (start 159.258 117.475) (end 159.258 114.2115) (width 0.5) (layer "F.Cu") (net 3))
@@
   (segment (start 112.546 85.045) (end 112.546 86.257) (width 0.35) (layer "F.Cu") (net 3))
   (segment (start 143.443 133.417) (end 143.764 133.096) (width 0.5) (layer "F.Cu") (net 3))
+  (segment (start 158.242 99.314) (end 159.893 100.965) (width 0.5) (layer "F.Cu") (net 3))
   (segment (start 153.147 137.795) (end 153.147 141.605) (width 2) (layer "F.Cu") (net 3))
   (segment (start 130.556 120.015) (end 126.974 120.015) (width 0.5) (layer "F.Cu") (net 3))
@@
   (segment (start 151.257 112.395) (end 148.336 112.395) (width 0.35) (layer "B.Cu") (net 37))
   (segment (start 162.179 113.792) (end 152.654 113.792) (width 0.35) (layer "B.Cu") (net 37))
+  (segment (start 158.242 92.07) (end 148.341 92.07) (width 0.5) (layer "F.Cu") (net 42))
+  (segment (start 148.341 92.07) (end 148.336 92.075) (width 0.5) (layer "F.Cu") (net 42))
   (segment (start 100.102 80.645) (end 102.846 80.645) (width 0.35) (layer "F.Cu") (net 52))
   (segment (start 156.49 107.3775) (end 156.4275 107.315) (width 0.5) (layer "F.Cu") (net 64))

Commit message: new model
Parts:
- added SW1: ARM, Connector_PinHeader_2.54mm:PinHeader_1x02_P2.54mm_Vertical, F.Cu at (122.6, 88.4)
Connections:
- U1 pad 5: unconnected-(U1-Pad5) -> /arm
Routing:
- net /arm: track 0.00 -> 6.04 mm
Changed lines of the file:
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@@
   (net 25 "/GPS_RX")
   (net 26 "Net-(R4-Pad2)")
-  (net 27 "unconnected-(U1-Pad5)")
+  (net 27 "Net-(J13-Pad1)")
   (net 28 "/PWM_SERVO1")
   (net 29 "/PWM_SERVO2")
@@
   (net 40 "unconnected-(U1-Pad31)")
   (net 41 "unconnected-(U1-Pad32)")
-  (net 42 "Net-(U1-Pad34)")
+  (net 42 "/arm")
   (net 43 "unconnected-(U1-Pad35)")
   (net 44 "unconnected-(U1-Pad37)")
@@
     (fp_line (start 1.27 -1.27) (end 1.27 3.81) (layer "F.Fab") (width 0.1))
     (pad "1" thru_hole rect (at 0 0) (size 1.7 1.7) (drill 1) (layers *.Cu *.Mask)
-      (net 42 "Net-(U1-Pad34)") (pinfunction "Pin_1") (pintype "passive"))
+      (net 27 "Net-(J13-Pad1)") (pinfunction "Pin_1") (pintype "passive"))
     (pad "2" thru_hole oval (at 0 2.54) (size 1.7 1.7) (drill 1) (layers *.Cu *.Mask)
       (net 3 "GND") (pinfunction "Pin_2") (pintype "passive"))
@@
       (net 66 "Net-(L1-Pad1)") (pintype "passive"))
     (model "${KICAD6_3DMODEL_DIR}/Resistor_SMD.3dshapes/R_1206_3216Metric.wrl"
+      (offset (xyz 0 0 0))
+      (scale (xyz 1 1 1))
+      (rotate (xyz 0 0 0))
+    )
+  )
+  (footprint "Connector_PinHeader_2.54mm:PinHeader_1x02_P2.54mm_Vertical" (layer "F.Cu")
+    (at 122.555 88.392 90)
+    (descr "Through hole straight pin header, 1x02, 2.54mm pitch, single row")
+    (tags "Through hole pin header THT 1x02 2.54mm single row")
+    (property "Sheetfile" "autopilot.kicad_sch")
+    (property "Sheetname" "")
+    (attr through_hole)
+    (fp_text reference "SW1" (at 0 -2.33 90) (layer "F.SilkS")
+      (effects (font (size 1 1) (thickness 0.15)))
+    )
+    (fp_text value "ARM" (at 0 4.87 90) (layer "F.Fab")
+      (effects (font (size 1 1) (thickness 0.15)))
+    )
+    (fp_text user "${REFERENCE}" (at 0 1.27) (layer "F.Fab")
+      (effects (font (size 1 1) (thickness 0.15)))
+    )
+    (fp_line (start -1.33 0) (end -1.33 -1.33) (layer "F.SilkS") (width 0.12))
+    (fp_line (start -1.33 -1.33) (end 0 -1.33) (layer "F.SilkS") (width 0.12))
+    (fp_line (start 1.33 1.27) (end 1.33 3.87) (layer "F.SilkS") (width 0.12))
+    (fp_line (start -1.33 1.27) (end 1.33 1.27) (layer "F.SilkS") (width 0.12))
+    (fp_line (start -1.33 1.27) (end -1.33 3.87) (layer "F.SilkS") (width 0.12))
+    (fp_line (start -1.33 3.87) (end 1.33 3.87) (layer "F.SilkS") (width 0.12))
+    (fp_line (start -1.8 4.35) (end 1.8 4.35) (layer "F.CrtYd") (width 0.05))
+    (fp_line (start 1.8 4.35) (end 1.8 -1.8) (layer "F.CrtYd") (width 0.05))
+    (fp_line (start -1.8 -1.8) (end -1.8 4.35) (layer "F.CrtYd") (width 0.05))
+    (fp_line (start 1.8 -1.8) (end -1.8 -1.8) (layer "F.CrtYd") (width 0.05))
+    (fp_line (start -1.27 -0.635) (end -0.635 -1.27) (layer "F.Fab") (width 0.1))
+    (fp_line (start 1.27 -1.27) (end 1.27 3.81) (layer "F.Fab") (width 0.1))
+    (fp_line (start -0.635 -1.27) (end 1.27 -1.27) (layer "F.Fab") (width 0.1))
+    (fp_line (start 1.27 3.81) (end -1.27 3.81) (layer "F.Fab") (width 0.1))
+    (fp_line (start -1.27 3.81) (end -1.27 -0.635) (layer "F.Fab") (width 0.1))
+    (pad "1" thru_hole rect (at 0 0 90) (size 1.7 1.7) (drill 1) (layers *.Cu *.Mask)
+      (net 3 "GND") (pintype "passive"))
+    (pad "2" thru_hole oval (at 0 2.54 90) (size 1.7 1.7) (drill 1) (layers *.Cu *.Mask)
+      (net 42 "/arm") (pintype "passive"))
+    (model "${KICAD6_3DMODEL_DIR}/Connector_PinHeader_2.54mm.3dshapes/PinHeader_1x02_P2.54mm_Vertical.wrl"
       (offset (xyz 0 0 0))
       (scale (xyz 1 1 1))
@@
       (net 12 "/GPS_RST") (pinfunction "GPIO2") (pintype "bidirectional"))
     (pad "5" thru_hole oval (at -8.89 -13.97) (size 1.7 1.7) (drill 1.02) (layers *.Cu *.Mask)
-      (net 27 "unconnected-(U1-Pad5)") (pinfunction "GPIO3") (pintype "bidirectional"))
+      (net 42 "/arm") (pinfunction "GPIO3") (pintype "bidirectional"))
     (pad "5" smd rect (at -8.89 -13.97) (size 3.5 1.7) (drill (offset -0.9 0)) (layers "F.Cu" "F.Mask")
-      (net 27 "unconnected-(U1-Pad5)") (pinfunction "GPIO3") (pintype "bidirectional"))
+      (net 42 "/arm") (pinfunction "GPIO3") (pintype "bidirectional"))
     (pad "6" thru_hole oval (at -8.89 -11.43) (size 1.7 1.7) (drill 1.02) (layers *.Cu *.Mask)
       (net 15 "/IMU_I2C_SDA") (pinfunction "GPIO4") (pintype "bidirectional"))
@@
       (net 3 "GND") (pinfunction "AGND") (pintype "power_in"))
     (pad "34" thru_hole oval (at 8.89 -8.89) (size 1.7 1.7) (drill 1.02) (layers *.Cu *.Mask)
-      (net 42 "Net-(U1-Pad34)") (pinfunction "GPIO28_ADC2") (pintype "bidirectional"))
+      (net 27 "Net-(J13-Pad1)") (pinfunction "GPIO28_ADC2") (pintype "bidirectional"))
     (pad "34" smd rect (at 8.89 -8.89) (size 3.5 1.7) (drill (offset 0.9 0)) (layers "F.Cu" "F.Mask")
-      (net 42 "Net-(U1-Pad34)") (pinfunction "GPIO28_ADC2") (pintype "bidirectional"))
+      (net 27 "Net-(J13-Pad1)") (pinfunction "GPIO28_ADC2") (pintype "bidirectional"))
     (pad "35" thru_hole oval (at 8.89 -11.43) (size 1.7 1.7) (drill 1.02) (layers *.Cu *.Mask)
       (net 43 "unconnected-(U1-Pad35)") (pinfunction "ADC_VREF") (pintype "power_in"))
@@
   (segment (start 118.364 97.663) (end 120.65 95.377) (width 0.35) (layer "F.Cu") (net 14))
   (segment (start 120.65 94.107) (end 122.682 92.075) (width 0.35) (layer "F.Cu") (net 14))
-  (segment (start 118.364 95.123) (end 123.952 89.535) (width 0.35) (layer "F.Cu") (net 15))
-  (segment (start 123.952 89.535) (end 130.556 89.535) (width 0.35) (layer "F.Cu") (net 15))
+  (segment (start 128.016 89.535) (end 130.556 89.535) (width 0.35) (layer "F.Cu") (net 15))
+  (segment (start 118.364 95.123) (end 122.301 91.186) (width 0.35) (layer "F.Cu") (net 15))
+  (segment (start 122.301 91.186) (end 126.365 91.186) (width 0.35) (layer "F.Cu") (net 15))
+  (segment (start 126.365 91.186) (end 128.016 89.535) (width 0.35) (layer "F.Cu") (net 15))
   (segment (start 123.952 99.949) (end 130.302 99.949) (width 0.25) (layer "F.Cu") (net 17))
   (segment (start 130.302 99.949) (end 130.556 99.695) (width 0.25) (layer "F.Cu") (net 17))
@@
   (segment (start 120.396 81.407) (end 118.958 82.845) (width 0.35) (layer "F.Cu") (net 26))
   (segment (start 122.91 76.835) (end 120.396 79.349) (width 0.35) (layer "F.Cu") (net 26))
+  (segment (start 158.242 92.07) (end 148.341 92.07) (width 0.5) (layer "F.Cu") (net 27))
+  (segment (start 148.341 92.07) (end 148.336 92.075) (width 0.5) (layer "F.Cu") (net 27))
   (segment (start 135.89 133.417) (end 135.130749 133.417) (width 0.35) (layer "F.Cu") (net 28))
   (segment (start 134.366 132.652251) (end 134.366 112.141) (width 0.35) (layer "F.Cu") (net 28))
@@
   (segment (start 151.257 112.395) (end 148.336 112.395) (width 0.35) (layer "B.Cu") (net 37))
   (segment (start 162.179 113.792) (end 152.654 113.792) (width 0.35) (layer "B.Cu") (net 37))
-  (segment (start 158.242 92.07) (end 148.341 92.07) (width 0.5) (layer "F.Cu") (net 42))
-  (segment (start 148.341 92.07) (end 148.336 92.075) (width 0.5) (layer "F.Cu") (net 42))
+  (segment (start 126.492 86.995) (end 125.095 88.392) (width 0.5) (layer "F.Cu") (net 42))
+  (segment (start 130.556 86.995) (end 126.492 86.995) (width 0.5) (layer "F.Cu") (net 42))
   (segment (start 100.102 80.645) (end 102.846 80.645) (width 0.35) (layer "F.Cu") (net 52))
   (segment (start 156.49 107.3775) (end 156.4275 107.315) (width 0.5) (layer "F.Cu") (net 64))
