File: electronics/mppt_boost/mppt.kicad_sch (KiCad schematic)
At the start: 49 parts, among them J1 I2C, J2 UART, J3 In, J4 In, J5 Out, J6 Out, Q1 IRLR2705TRPBF, Q2 IRLR2705TRPBF, SW1 SW_DIP_x01, U1 AD8211, U2 AD8211, U3 ATmega328P-A, U4 2EDN852x, U5 L78L15_SO8, Y1 16.00M-SMDHC49S

Commit message: 3d renders of electronics
Parts:
- added R14: 10k, Resistor_SMD:R_1206_3216Metric_Pad1.30x1.75mm_HandSolder, symbol Device:R
Connections:
- net +5V: now also U3.18 (AVCC), R14.1
- net at SW1.1, U3.29 (~{RESET}/PC6): now also R14.2
Other:
- moved on the sheet: SW1
Changed lines of the file:
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@@
   (junction (at 80.01 129.54) (diameter 0) (color 0 0 0 0)
   )
+  (junction (at 196.85 29.21) (diameter 0) (color 0 0 0 0)
+  )
   (junction (at 152.4 81.28) (diameter 0) (color 0 0 0 0)
   )
@@
   (junction (at 153.67 152.4) (diameter 0) (color 0 0 0 0)
   )
+  (junction (at 231.14 80.01) (diameter 0) (color 0 0 0 0)
+  )
   (junction (at 222.25 55.88) (diameter 0) (color 0 0 0 0)
   )
@@
     (stroke (width 0) (type default) (color 0 0 0 0))
   )
+  (wire (pts (xy 232.41 80.01) (xy 231.14 80.01))
+    (stroke (width 0) (type default) (color 0 0 0 0))
+  )
   (wire (pts (xy 25.4 139.7) (xy 25.4 129.54))
     (stroke (width 0) (type default) (color 0 0 0 0))
@@
     (stroke (width 0) (type default) (color 0 0 0 0))
   )
+  (wire (pts (xy 248.92 80.01) (xy 248.92 83.82))
+    (stroke (width 0) (type default) (color 0 0 0 0))
+  )
   (wire (pts (xy 102.87 58.42) (xy 86.36 58.42))
     (stroke (width 0) (type default) (color 0 0 0 0))
@@
     (stroke (width 0) (type default) (color 0 0 0 0))
   )
+  (wire (pts (xy 199.39 34.29) (xy 199.39 29.21))
+    (stroke (width 0) (type default) (color 0 0 0 0))
+  )
   (wire (pts (xy 22.86 139.7) (xy 25.4 139.7))
     (stroke (width 0) (type default) (color 0 0 0 0))
@@
     (stroke (width 0) (type default) (color 0 0 0 0))
   )
-  (wire (pts (xy 246.38 83.82) (xy 246.38 80.01))
-    (stroke (width 0) (type default) (color 0 0 0 0))
-  )
   (wire (pts (xy 104.14 143.51) (xy 104.14 152.4))
     (stroke (width 0) (type default) (color 0 0 0 0))
@@
     (stroke (width 0) (type default) (color 0 0 0 0))
   )
+  (wire (pts (xy 247.65 80.01) (xy 248.92 80.01))
+    (stroke (width 0) (type default) (color 0 0 0 0))
+  )
   (wire (pts (xy 152.4 81.28) (xy 170.18 81.28))
     (stroke (width 0) (type default) (color 0 0 0 0))
@@
     (stroke (width 0) (type default) (color 0 0 0 0))
   )
+  (wire (pts (xy 199.39 29.21) (xy 196.85 29.21))
+    (stroke (width 0) (type default) (color 0 0 0 0))
+  )
+  (wire (pts (xy 231.14 83.82) (xy 231.14 80.01))
+    (stroke (width 0) (type default) (color 0 0 0 0))
+  )
   (wire (pts (xy 152.4 58.42) (xy 170.18 58.42))
     (stroke (width 0) (type default) (color 0 0 0 0))
@@
     (stroke (width 0) (type default) (color 0 0 0 0))
   )
-  (wire (pts (xy 212.09 80.01) (xy 229.87 80.01))
+  (wire (pts (xy 212.09 80.01) (xy 231.14 80.01))
     (stroke (width 0) (type default) (color 0 0 0 0))
   )
@@
     (stroke (width 0) (type default) (color 0 0 0 0))
   )
-  (wire (pts (xy 246.38 80.01) (xy 245.11 80.01))
-    (stroke (width 0) (type default) (color 0 0 0 0))
-  )
   (wire (pts (xy 78.74 48.26) (xy 78.74 39.37))
     (stroke (width 0) (type default) (color 0 0 0 0))
@@
   )
   (wire (pts (xy 22.86 142.24) (xy 25.4 142.24))
+    (stroke (width 0) (type default) (color 0 0 0 0))
+  )
+  (wire (pts (xy 231.14 91.44) (xy 240.03 91.44))
     (stroke (width 0) (type default) (color 0 0 0 0))
   )
@@
     (pin "1")
   )
-  (symbol (lib_id "power:GND") (at 246.38 83.82 0) (unit 1)
-    (in_bom yes) (on_board yes) (fields_autoplaced)
-    (property "Reference" "#PWR017" (id 0) (at 246.38 90.17 0)
-      (effects (font (size 1.27 1.27)) hide)
-    )
-    (property "Value" "GND" (id 1) (at 246.38 88.9 0))
-    (property "Footprint" "" (id 2) (at 246.38 83.82 0)
-      (effects (font (size 1.27 1.27)) hide)
-    )
-    (property "Datasheet" "" (id 3) (at 246.38 83.82 0)
+  (symbol (lib_id "power:GND") (at 248.92 83.82 0) (unit 1)
+    (in_bom yes) (on_board yes) (fields_autoplaced)
+    (property "Reference" "#PWR017" (id 0) (at 248.92 90.17 0)
+      (effects (font (size 1.27 1.27)) hide)
+    )
+    (property "Value" "GND" (id 1) (at 248.92 88.9 0))
+    (property "Footprint" "" (id 2) (at 248.92 83.82 0)
+      (effects (font (size 1.27 1.27)) hide)
+    )
+    (property "Datasheet" "" (id 3) (at 248.92 83.82 0)
       (effects (font (size 1.27 1.27)) hide)
     )
@@
     (pin "1")
     (pin "2")
+  )
+  (symbol (lib_id "Device:R") (at 231.14 87.63 180) (unit 1)
+    (in_bom yes) (on_board yes) (fields_autoplaced)
+    (property "Reference" "R14" (id 0) (at 233.68 86.3599 0)
+      (effects (font (size 1.27 1.27)) (justify right))
+    )
+    (property "Value" "10k" (id 1) (at 233.68 88.8999 0)
+      (effects (font (size 1.27 1.27)) (justify right))
+    )
+    (property "Footprint" "Resistor_SMD:R_1206_3216Metric_Pad1.30x1.75mm_HandSolder" (id 2) (at 232.918 87.63 90)
+      (effects (font (size 1.27 1.27)) hide)
+    )
+    (property "Datasheet" "~" (id 3) (at 231.14 87.63 0)
+      (effects (font (size 1.27 1.27)) hide)
+    )
+    (pin "1")
+    (pin "2")
+  )
+  (symbol (lib_id "power:+5V") (at 240.03 91.44 0) (unit 1)
+    (in_bom yes) (on_board yes) (fields_autoplaced)
+    (property "Reference" "#PWR0104" (id 0) (at 240.03 95.25 0)
+      (effects (font (size 1.27 1.27)) hide)
+    )
+    (property "Value" "+5V" (id 1) (at 240.03 86.36 0))
+    (property "Footprint" "" (id 2) (at 240.03 91.44 0)
+      (effects (font (size 1.27 1.27)) hide)
+    )
+    (property "Datasheet" "" (id 3) (at 240.03 91.44 0)
+      (effects (font (size 1.27 1.27)) hide)
+    )
+    (pin "1")
   )
   (symbol (lib_id "Device:R") (at 153.67 146.05 180) (unit 1)
@@
     (pin "1")
   )
-  (symbol (lib_id "Switch:SW_DIP_x01") (at 237.49 80.01 0) (unit 1)
-    (in_bom yes) (on_board yes) (fields_autoplaced)
-    (property "Reference" "SW1" (id 0) (at 237.49 72.39 0))
-    (property "Value" "SW_DIP_x01" (id 1) (at 237.49 74.93 0))
-    (property "Footprint" "Jumper:SolderJumper-2_P1.3mm_Open_RoundedPad1.0x1.5mm" (id 2) (at 237.49 80.01 0)
-      (effects (font (size 1.27 1.27)) hide)
-    )
-    (property "Datasheet" "~" (id 3) (at 237.49 80.01 0)
+  (symbol (lib_id "Switch:SW_DIP_x01") (at 240.03 80.01 0) (unit 1)
+    (in_bom yes) (on_board yes) (fields_autoplaced)
+    (property "Reference" "SW1" (id 0) (at 240.03 72.39 0))
+    (property "Value" "SW_DIP_x01" (id 1) (at 240.03 74.93 0))
+    (property "Footprint" "Jumper:SolderJumper-2_P1.3mm_Open_RoundedPad1.0x1.5mm" (id 2) (at 240.03 80.01 0)
+      (effects (font (size 1.27 1.27)) hide)
+    )
+    (property "Datasheet" "~" (id 3) (at 240.03 80.01 0)
       (effects (font (size 1.27 1.27)) hide)
     )
@@
       (reference "#PWR0103") (unit 1) (value "GND2") (footprint "")
     )
+    (path "/0caa6f73-b1a3-4287-a615-1a082042887d"
+      (reference "#PWR0104") (unit 1) (value "+5V") (footprint "")
+    )
     (path "/47ae361a-4310-4583-826d-5c506796dca5"
       (reference "C1") (unit 1) (value "10u") (footprint "Capacitor_Tantalum_SMD:CP_EIA-7343-15_Kemet-W_Pad2.25x2.55mm_HandSolder")
@@
       (reference "R13") (unit 1) (value "100k") (footprint "Resistor_SMD:R_1206_3216Metric_Pad1.30x1.75mm_HandSolder")
     )
+    (path "/0c3c226b-48b5-4c31-8f40-0b66529e70ce"
+      (reference "R14") (unit 1) (value "10k") (footprint "Resistor_SMD:R_1206_3216Metric_Pad1.30x1.75mm_HandSolder")
+    )
     (path "/d39a6313-1ab9-4ec3-80c7-c6ab9bb1690b"
