File: electronics/mppt_boost/mppt.kicad_pcb (KiCad board)
At the start: 2 copper layers, 63 x 71.9 mm, 49 parts, among them J1 I2C, J2 UART, J3 In, J4 In, J5 Out, J6 Out, Q1 IRLR2705TRPBF, Q2 IRLR2705TRPBF, SW1 SW_DIP_x01, U1 AD8211, U2 AD8211, U3 ATmega328P-A, U4 2EDN852x, U5 L78L15_SO8, Y1 16.00M-SMDHC49S

Commit message: 3d renders of electronics
Parts:
- added R14: 10k, Resistor_SMD:R_1206_3216Metric_Pad1.30x1.75mm_HandSolder, F.Cu at (123.3, 109.7)
Connections:
- U3 pad 18: unconnected-(U3-Pad18) -> +5V
Routing:
- net +5V: track 203.5 -> 210.8 mm
- net Net-(SW1-Pad1): track 32.9 -> 37.4 mm
