File: electronics/power_board/power_board.kicad_pcb (KiCad board)
At the start: 2 copper layers, 43 parts, among them J1 Vin, J2 I2C_low, J3 I2C_high, J4 3.3V out, J5 5V out, Q1 2N7002E, Q2 2N7002E, U1 TPS54228, U2 TPS54228

Commit message: power board finished
Parts:
- removed J2: I2C_low, Connector_PinSocket_2.54mm:PinSocket_1x03_P2.54mm_Vertical
- removed J3: I2C_high, Connector_PinSocket_2.54mm:PinSocket_1x03_P2.54mm_Vertical
- removed Q1, Q2: 2N7002E, Package_TO_SOT_SMD:SOT-23
- removed R10, R3, R8, R9: 10k, Resistor_SMD:R_1206_3216Metric_Pad1.30x1.75mm_HandSolder
- added J7: Vin, moje:ARK, F.Cu at (143.6, 58.5)
- added R13: 4.7k, Resistor_SMD:R_1206_3216Metric_Pad1.30x1.75mm_HandSolder, F.Cu at (118.1, 31.9)
- added R16: 4.7k, Resistor_SMD:R_1206_3216Metric_Pad1.30x1.75mm_HandSolder, F.Cu at (159.6, 50.4)
- C15, C16, C17, C18: value 22p -> 22u; footprint Capacitor_SMD:C_1206_3216Metric_Pad1.33x1.80mm_HandSolder -> Capacitor_SMD:CP_Elec_6.3x5.4
- R1: value 73.2k -> 68k
- R2: value 124k -> 120k
- moved C6 71.7 mm to (157.1, 45.3), turned to -90 degrees
- moved R1 71.5 mm to (119.4, 27.9), turned to 180 degrees
- moved C2 69.9 mm to (157.1, 54.4), turned to 90 degrees
- moved D2 67.5 mm to (142.5, 24.6)
- moved C9 65.7 mm to (127.1, 27.7)
- moved C11 63.6 mm to (127.1, 30.1)
- moved C3 61.8 mm to (127.1, 25.3)
- moved C13 58.1 mm to (132.3, 33.2), turned to 90 degrees
- moved L1 57.6 mm to (141.5, 34.7)
- moved R12 57.2 mm to (147.8, 24.6), turned to 180 degrees
- moved J5 56.2 mm to (118.6, 46.7), turned to 90 degrees
- moved L2 54.9 mm to (137.2, 48.6), turned to 180 degrees
- moved J4 54.4 mm to (159.5, 37.2), turned to -90 degrees
- moved C17 54.0 mm to (154.2, 28.2), turned to 180 degrees
- moved R4 53.3 mm to (118.1, 37.0), turned to 90 degrees
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Connections:
- C10 pad 2: VBUS -> VAA
- C11 pad 2: VBUS -> VCC
- C12 pad 2: VBUS -> VAA
- C3 pad 2: VBUS -> VCC
- C4 pad 2: VBUS -> VAA
- C9 pad 2: VBUS -> VCC
- J1 pad 1: VBUS -> VCC
- R1 pad 2: Net-(C1-Pad2) -> Net-(R1-Pad2)
- R2 pad 2: Net-(C2-Pad2) -> Net-(R2-Pad2)
- R6 pad 1: VBUS -> VCC
- R7 pad 1: VBUS -> VAA
- U1 pad 5: Net-(U1-Pad) -> GND
- U1 pad 8: VBUS -> VCC
- U1 pad 9: (no net) -> GND
- U2 pad 5: Net-(U2-Pad) -> GND
- U2 pad 8: VBUS -> VAA
- U2 pad 9: (no net) -> GND
Routing:
- net GND: track 0.00 -> 193.0 mm
- net +3.3V: track 0.00 -> 67.3 mm
- net +5V: track 0.00 -> 66.5 mm
- net VCC: track 0.00 -> 19.9 mm
- net VAA: track 0.00 -> 19.7 mm
- net Net-(C2-Pad2): track 0.00 -> 10.7 mm
- net Net-(C13-Pad1): track 0.00 -> 7.31 mm
- net Net-(C14-Pad1): track 0.00 -> 6.61 mm
- net Net-(C13-Pad2): track 0.00 -> 5.14 mm
- net Net-(C1-Pad2): track 0.00 -> 4.89 mm
- net Net-(C14-Pad2): track 0.00 -> 4.08 mm
- net Net-(C6-Pad2): track 0.00 -> 3.74 mm
- net Net-(C5-Pad2): track 0.00 -> 2.64 mm
- net Net-(R1-Pad2): track 0.00 -> 2.50 mm
- net Net-(C8-Pad2): track 0.00 -> 2.31 mm
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Other:
- board outline added: 44.5 x 39.4 mm

Commit message: 3d renders of electronics
Routing:
- net Net-(C1-Pad2): track 4.89 -> 7.31 mm
Changed lines of the file:
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@@
+      (rotate (xyz 0 0 0))
+    )
+    (model "${KICAD6_3DMODEL_DIR}/Inductor_SMD.3dshapes/L_TDK_SLF12575.wrl"
+      (offset (xyz 0 0 0))
+      (scale (xyz 1 1 1))
       (rotate (xyz 0 0 0))
     )
@@
       (rotate (xyz 0 0 0))
     )
+    (model "${KICAD6_3DMODEL_DIR}/Inductor_SMD.3dshapes/L_TDK_SLF12575.wrl"
+      (offset (xyz 0 0 0))
+      (scale (xyz 1 1 1))
+      (rotate (xyz 0 0 0))
+    )
   )
   (footprint "moje:ARK" (layer "F.Cu")
@@
   (segment (start 123.3471 33.4395) (end 123.4102 33.5026) (width 0.5) (layer "F.Cu") (net 2))
   (segment (start 120.523 33.4395) (end 123.3471 33.4395) (width 0.5) (layer "F.Cu") (net 2))
+  (segment (start 118.11 33.427) (end 120.5105 33.427) (width 0.5) (layer "F.Cu") (net 2))
+  (segment (start 120.5105 33.427) (end 120.523 33.4395) (width 0.5) (layer "F.Cu") (net 2))
   (segment (start 118.11 35.407) (end 118.11 33.427) (width 0.5) (layer "F.Cu") (net 2))
   (segment (start 120.009 55.245) (end 120.009 50.6035) (width 2) (layer "F.Cu") (net 3))
